Commit message: adding RigidBodyDynamics pure script and some more urdfs relating to bsm

File: urdf_parser/urdfs/bsm_2thread_nohanger.urdf (robot description, URDF)
Before this commit: robot BranchScissorMechanism, 33 links, 32 joints
Links:
- removed link arm1-2-1
- removed link arm1-2-2
- removed link arm1-4-1
- removed link arm1-4-2
- removed link base_link
- removed link hand1-2
- removed link hand1-4
- removed link hand2-1
- removed link hand2-2
- removed link hand2-3
- removed link hand2-4
- link arm1-1-1: geometry visual cylinder length=0.080948 radius=0.0059505
- link arm1-1-2: geometry visual cylinder length=0.080948 radius=0.0059505
- link arm1-3-1: geometry visual cylinder length=0.080948 radius=0.0059505
- link arm1-3-2: geometry visual cylinder length=0.080948 radius=0.0059505
- link arm2-1-1: geometry visual cylinder length=0.080948 radius=0.0059505
- link arm2-1-2: geometry visual cylinder length=0.080948 radius=0.0059505
- link arm2-2-1: geometry visual cylinder length=0.080948 radius=0.0059505
- link arm2-2-2: geometry visual cylinder length=0.080948 radius=0.0059505
- link arm2-3-1: geometry visual cylinder length=0.080948 radius=0.0059505
- link arm2-3-2: geometry visual cylinder length=0.080948 radius=0.0059505
- link arm2-4-1: geometry visual cylinder length=0.080948 radius=0.0059505
- link arm2-4-2: geometry visual cylinder length=0.080948 radius=0.0059505
- link four1-1: geometry visual cylinder length=0.017 radius=0.005
- link four1-2: geometry visual cylinder length=0.017 radius=0.005
- link four1-3: geometry visual cylinder length=0.017 radius=0.005
- link four1-4: geometry visual cylinder length=0.017 radius=0.005
- link four2-1: geometry visual cylinder length=0.017 radius=0.005
- link four2-2: geometry visual cylinder length=0.017 radius=0.005
- link four2-3: geometry visual cylinder length=0.017 radius=0.005
- link four2-4: geometry visual cylinder length=0.017 radius=0.005
- link hand1-1: geometry visual cylinder length=0.034 radius=0.008
- link hand1-3: geometry visual cylinder length=0.034 radius=0.008
Joints:
- removed joint arm1-2
- removed joint arm1-4
- removed joint bsm1-to-bsm2
- removed joint hand1-2
- removed joint hand1-4
- removed joint hand2-1
- removed joint hand2-2
- removed joint hand2-3
- removed joint hand2-4
- removed joint world
- removed joint wrist1-2
- removed joint wrist1-4
- added joint arm2-3-1-to-hand1-1: type continuous, parent arm2-3-1, child hand1-1, origin xyz=0.06309 0 -0.050716 rpy=0 0 3.14159265359, axis 0 1 0
- joint arm1-1: axis 0 1 0 -> (none); child arm1-1-2 -> arm1-1-1; origin xyz=0 0 0 rpy=0 0 0 -> xyz=0.06309 0 -0.050716 rpy=0 0 0; parent arm1-1-1 -> arm1-1-2
- joint arm2-1: child arm2-1-2 -> arm2-1-1; origin xyz=0 0 0 rpy=0 0 0 -> xyz=0.06309 0 -0.050716 rpy=0 0 0; parent arm2-1-1 -> arm2-1-2
- joint four1-1-to-four1-2: origin xyz=-0.017 -0.017 0 rpy=0 0 1.5708 -> xyz=-0.017 -0.017 0 rpy=0 0 1.57079632679
- joint four1-1-to-four1-3: origin xyz=0 -0.034 0 rpy=0 0 3.1416 -> xyz=0 -0.034 0 rpy=0 0 3.14159265359
- joint four1-1-to-four1-4: origin xyz=0.017 -0.017 0 rpy=0 0 -1.5708 -> xyz=0.017 -0.017 0 rpy=0 0 -1.57079632679
- joint four2-1-to-four2-2: origin xyz=-0.017 -0.017 0 rpy=0 0 1.5708 -> xyz=-0.017 -0.017 0 rpy=0 0 1.57079632679
- joint four2-1-to-four2-3: origin xyz=0 -0.034 0 rpy=0 0 3.1416 -> xyz=0 -0.034 0 rpy=0 0 3.14159265359
- joint four2-1-to-four2-4: origin xyz=0.017 -0.017 0 rpy=0 0 -1.5708 -> xyz=0.017 -0.017 0 rpy=0 0 -1.57079632679
- joint hand1-1: child hand1-1 -> arm1-1-2; origin xyz=-0.06309 0 0.050716 rpy=0 0 0 -> xyz=0 0.034 0 rpy=0 0 0; parent arm1-1-2 -> hand1-1
- joint wrist1-1: axis (none) -> 0 1 0; child arm1-1-1 -> four1-1; parent four1-1 -> arm1-1-1
- joint wrist1-3: axis (none) -> 0 1 0
- joint wrist2-1: axis (none) -> 0 1 0; child arm2-1-1 -> four2-1; parent four2-1 -> arm2-1-1; type continuous -> fixed
- joint wrist2-2: axis (none) -> 0 1 0
- joint wrist2-3: axis (none) -> 0 1 0
- joint wrist2-4: axis (none) -> 0 1 0

File: urdf_parser/urdfs/bsm_new.urdf (robot description, URDF)
Before this commit: robot BranchScissorMechanism, 33 links, 32 joints
Links:
- added link hanger-1, mass 1; visual cylinder length=0.017 radius=0.0059505
- added link hanger-3, mass 1; visual cylinder length=0.017 radius=0.0059505
- added link string-1, mass 1; visual cylinder length=0.071468 radius=0.0059505
- added link string-3, mass 1; visual cylinder length=0.071468 radius=0.0059505
- link arm1-1-1: geometry visual cylinder length=0.080948 radius=0.0059505
- link arm1-1-2: geometry visual cylinder length=0.080948 radius=0.0059505
- link arm1-2-1: geometry visual cylinder length=0.080948 radius=0.0059505
- link arm1-2-2: geometry visual cylinder length=0.080948 radius=0.0059505
- link arm1-3-1: geometry visual cylinder length=0.080948 radius=0.0059505
- link arm1-3-2: geometry visual cylinder length=0.080948 radius=0.0059505
- link arm1-4-1: geometry visual cylinder length=0.080948 radius=0.0059505
- link arm1-4-2: geometry visual cylinder length=0.080948 radius=0.0059505
- link arm2-1-1: geometry visual cylinder length=0.080948 radius=0.0059505
- link arm2-1-2: geometry visual cylinder length=0.080948 radius=0.0059505
- link arm2-2-1: geometry visual cylinder length=0.080948 radius=0.0059505
- link arm2-2-2: geometry visual cylinder length=0.080948 radius=0.0059505
- link arm2-3-1: geometry visual cylinder length=0.080948 radius=0.0059505
- link arm2-3-2: geometry visual cylinder length=0.080948 radius=0.0059505
- link arm2-4-1: geometry visual cylinder length=0.080948 radius=0.0059505
- link arm2-4-2: geometry visual cylinder length=0.080948 radius=0.0059505
- link four1-1: geometry visual cylinder length=0.017 radius=0.005
- link four1-2: geometry visual cylinder length=0.017 radius=0.005
- link four1-3: geometry visual cylinder length=0.017 radius=0.005
- link four1-4: geometry visual cylinder length=0.017 radius=0.005
- link four2-1: geometry visual cylinder length=0.017 radius=0.005
- link four2-2: geometry visual cylinder length=0.017 radius=0.005
- link four2-3: geometry visual cylinder length=0.017 radius=0.005
- link four2-4: geometry visual cylinder length=0.017 radius=0.005
- link hand1-1: geometry visual cylinder length=0.034 radius=0.008
- link hand1-2: geometry visual cylinder length=0.034 radius=0.008
- link hand1-3: geometry visual cylinder length=0.034 radius=0.008
- link hand1-4: geometry visual cylinder length=0.034 radius=0.008
- link hand2-1: geometry visual cylinder length=0.034 radius=0.008
- link hand2-2: geometry visual cylinder length=0.034 radius=0.008
- link hand2-3: geometry visual cylinder length=0.034 radius=0.008
- link hand2-4: geometry visual cylinder length=0.034 radius=0.008
Joints:
- removed joint bsm1-to-bsm2
- removed joint world
- added joint arm2-3-1-to-hand1-1: type continuous, parent arm2-3-1, child hand1-1, origin xyz=0.06309 0 -0.050716 rpy=0 0 3.14159265358979323846, axis 0 1 0
- added joint hand-to-string-3: type continuous, parent hand2-3, child string-3, origin xyz=0 -0.034 0 rpy=0 0 0, axis 0 1 0
- added joint hanger-1: type fixed, parent base_link, child hanger-1, origin xyz=0 0 0 rpy=0 0 0
- added joint hanger-3: type fixed, parent base_link, child hanger-3, origin xyz=0 0 0 rpy=0 0 3.14159265358979323846
- added joint string-1: type continuous, parent hanger-1, child string-1, origin xyz=0 -0.017 0 rpy=0 0 0, axis 0 1 0
- added joint string-to-hand-1: type continuous, parent string-1, child hand2-1, origin xyz=-0.06309 0 -0.033576 rpy=0 0 0, axis 0 1 0
- joint arm1-1: axis 0 1 0 -> (none); child arm1-1-2 -> arm1-1-1; origin xyz=0 0 0 rpy=0 0 0 -> xyz=0.06309 0 -0.050716 rpy=0 0 0; parent arm1-1-1 -> arm1-1-2
- joint arm2-1: child arm2-1-2 -> arm2-1-1; origin xyz=0 0 0 rpy=0 0 0 -> xyz=0.06309 0 -0.050716 rpy=0 0 0; parent arm2-1-1 -> arm2-1-2
- joint four1-1-to-four1-2: origin xyz=-0.017 -0.017 0 rpy=0 0 1.5708 -> xyz=-0.017 -0.017 0 rpy=0 0 1.570796326794897
- joint four1-1-to-four1-3: origin xyz=0 -0.034 0 rpy=0 0 3.1416 -> xyz=0 -0.034 0 rpy=0 0 3.14159265358979323846
- joint four1-1-to-four1-4: origin xyz=0.017 -0.017 0 rpy=0 0 -1.5708 -> xyz=0.017 -0.017 0 rpy=0 0 -1.570796326794897
- joint four2-1-to-four2-2: origin xyz=-0.017 -0.017 0 rpy=0 0 1.5708 -> xyz=-0.017 -0.017 0 rpy=0 0 1.570796326794897
- joint four2-1-to-four2-3: origin xyz=0 -0.034 0 rpy=0 0 3.1416 -> xyz=0 -0.034 0 rpy=0 0 3.14159265358979323846
- joint four2-1-to-four2-4: origin xyz=0.017 -0.017 0 rpy=0 0 -1.5708 -> xyz=0.017 -0.017 0 rpy=0 0 -1.570796326794897
- joint hand1-1: child hand1-1 -> arm1-1-2; origin xyz=-0.06309 0 0.050716 rpy=0 0 0 -> xyz=0 0.034 0 rpy=0 0 0; parent arm1-1-2 -> hand1-1
- joint hand2-1: child hand2-1 -> arm2-1-2; origin xyz=-0.06309 0 0.050716 rpy=0 0 0 -> xyz=0 0.034 0 rpy=0 0 0; parent arm2-1-2 -> hand2-1
- joint wrist1-1: axis (none) -> 0 1 0; child arm1-1-1 -> four1-1; parent four1-1 -> arm1-1-1
- joint wrist1-2: axis (none) -> 0 1 0
- joint wrist1-3: axis (none) -> 0 1 0
- joint wrist1-4: axis (none) -> 0 1 0
- joint wrist2-1: axis (none) -> 0 1 0; child arm2-1-1 -> four2-1; parent four2-1 -> arm2-1-1; type continuous -> fixed
- joint wrist2-2: axis (none) -> 0 1 0
- joint wrist2-3: axis (none) -> 0 1 0
- joint wrist2-4: axis (none) -> 0 1 0

File: urdf_parser/urdfs/bsm_new_2thread.urdf (robot description, URDF)
Before this commit: robot BranchScissorMechanism, 33 links, 32 joints
Links:
- removed link arm1-2-1
- removed link arm1-2-2
- removed link arm1-4-1
- removed link arm1-4-2
- removed link hand1-2
- removed link hand1-4
- added link hanger-1, mass 1; visual cylinder length=0.017 radius=0.0059505
- added link hanger-3, mass 1; visual cylinder length=0.017 radius=0.0059505
- added link string-1, mass 1; visual cylinder length=0.071468 radius=0.0059505
- added link string-3, mass 1; visual cylinder length=0.071468 radius=0.0059505
- link arm1-1-1: geometry visual cylinder length=0.080948 radius=0.0059505
- link arm1-1-2: geometry visual cylinder length=0.080948 radius=0.0059505
- link arm1-3-1: geometry visual cylinder length=0.080948 radius=0.0059505
- link arm1-3-2: geometry visual cylinder length=0.080948 radius=0.0059505
- link arm2-1-1: geometry visual cylinder length=0.080948 radius=0.0059505
- link arm2-1-2: geometry visual cylinder length=0.080948 radius=0.0059505
- link arm2-2-1: geometry visual cylinder length=0.080948 radius=0.0059505
- link arm2-2-2: geometry visual cylinder length=0.080948 radius=0.0059505
- link arm2-3-1: geometry visual cylinder length=0.080948 radius=0.0059505
- link arm2-3-2: geometry visual cylinder length=0.080948 radius=0.0059505
- link arm2-4-1: geometry visual cylinder length=0.080948 radius=0.0059505
- link arm2-4-2: geometry visual cylinder length=0.080948 radius=0.0059505
- link four1-1: geometry visual cylinder length=0.017 radius=0.005
- link four1-2: geometry visual cylinder length=0.017 radius=0.005
- link four1-3: geometry visual cylinder length=0.017 radius=0.005
- link four1-4: geometry visual cylinder length=0.017 radius=0.005
- link four2-1: geometry visual cylinder length=0.017 radius=0.005
- link four2-2: geometry visual cylinder length=0.017 radius=0.005
- link four2-3: geometry visual cylinder length=0.017 radius=0.005
- link four2-4: geometry visual cylinder length=0.017 radius=0.005
- link hand1-1: geometry visual cylinder length=0.034 radius=0.008
- link hand1-3: geometry visual cylinder length=0.034 radius=0.008
- link hand2-1: geometry visual cylinder length=0.034 radius=0.008
- link hand2-2: geometry visual cylinder length=0.034 radius=0.008
- link hand2-3: geometry visual cylinder length=0.034 radius=0.008
- link hand2-4: geometry visual cylinder length=0.034 radius=0.008
Joints:
- removed joint arm1-2
- removed joint arm1-4
- removed joint bsm1-to-bsm2
- removed joint hand1-2
- removed joint hand1-4
- removed joint world
- removed joint wrist1-2
- removed joint wrist1-4
- added joint arm2-3-1-to-hand1-1: type continuous, parent arm2-3-1, child hand1-1, origin xyz=0.06309 0 -0.050716 rpy=0 0 3.14159265359, axis 0 1 0
- added joint hand-to-string-3: type continuous, parent hand2-3, child string-3, origin xyz=0 -0.034 0 rpy=0 0 0, axis 0 1 0
- added joint hanger-1: type fixed, parent base_link, child hanger-1, origin xyz=0 0 0 rpy=0 0 0
- added joint hanger-3: type fixed, parent base_link, child hanger-3, origin xyz=0 0 0 rpy=0 0 3.14159
- added joint string-1: type continuous, parent hanger-1, child string-1, origin xyz=0 -0.017 0 rpy=0 0 0, axis 0 1 0
- added joint string-to-hand-1: type continuous, parent string-1, child hand2-1, origin xyz=-0.06309 0 -0.033576 rpy=0 0 0, axis 0 1 0
- joint arm1-1: axis 0 1 0 -> (none); child arm1-1-2 -> arm1-1-1; origin xyz=0 0 0 rpy=0 0 0 -> xyz=0.06309 0 -0.050716 rpy=0 0 0; parent arm1-1-1 -> arm1-1-2
- joint arm2-1: child arm2-1-2 -> arm2-1-1; origin xyz=0 0 0 rpy=0 0 0 -> xyz=0.06309 0 -0.050716 rpy=0 0 0; parent arm2-1-1 -> arm2-1-2
- joint four1-1-to-four1-2: origin xyz=-0.017 -0.017 0 rpy=0 0 1.5708 -> xyz=-0.017 -0.017 0 rpy=0 0 1.57079632679
- joint four1-1-to-four1-3: origin xyz=0 -0.034 0 rpy=0 0 3.1416 -> xyz=0 -0.034 0 rpy=0 0 3.14159265359
- joint four1-1-to-four1-4: origin xyz=0.017 -0.017 0 rpy=0 0 -1.5708 -> xyz=0.017 -0.017 0 rpy=0 0 -1.57079632679
- joint four2-1-to-four2-2: origin xyz=-0.017 -0.017 0 rpy=0 0 1.5708 -> xyz=-0.017 -0.017 0 rpy=0 0 1.57079632679
- joint four2-1-to-four2-3: origin xyz=0 -0.034 0 rpy=0 0 3.1416 -> xyz=0 -0.034 0 rpy=0 0 3.14159265359
- joint four2-1-to-four2-4: origin xyz=0.017 -0.017 0 rpy=0 0 -1.5708 -> xyz=0.017 -0.017 0 rpy=0 0 -1.57079632679
- joint hand1-1: child hand1-1 -> arm1-1-2; origin xyz=-0.06309 0 0.050716 rpy=0 0 0 -> xyz=0 0.034 0 rpy=0 0 0; parent arm1-1-2 -> hand1-1
- joint hand2-1: child hand2-1 -> arm2-1-2; origin xyz=-0.06309 0 0.050716 rpy=0 0 0 -> xyz=0 0.034 0 rpy=0 0 0; parent arm2-1-2 -> hand2-1
- joint wrist1-1: axis (none) -> 0 1 0; child arm1-1-1 -> four1-1; parent four1-1 -> arm1-1-1
- joint wrist1-3: axis (none) -> 0 1 0
- joint wrist2-1: axis (none) -> 0 1 0; child arm2-1-1 -> four2-1; parent four2-1 -> arm2-1-1; type continuous -> fixed
- joint wrist2-2: axis (none) -> 0 1 0
- joint wrist2-3: axis (none) -> 0 1 0
- joint wrist2-4: axis (none) -> 0 1 0

File: urdf_parser/urdfs/bsm_nohanger.urdf (robot description, URDF)
Before this commit: robot BranchScissorMechanism, 33 links, 32 joints
Links:
- removed link base_link
- removed link hand2-1
- removed link hand2-2
- removed link hand2-3
- removed link hand2-4
- link arm1-1-1: geometry visual cylinder length=0.080948 radius=0.0059505
- link arm1-1-2: geometry visual cylinder length=0.080948 radius=0.0059505
- link arm1-2-1: geometry visual cylinder length=0.080948 radius=0.0059505
- link arm1-2-2: geometry visual cylinder length=0.080948 radius=0.0059505
- link arm1-3-1: geometry visual cylinder length=0.080948 radius=0.0059505
- link arm1-3-2: geometry visual cylinder length=0.080948 radius=0.0059505
- link arm1-4-1: geometry visual cylinder length=0.080948 radius=0.0059505
- link arm1-4-2: geometry visual cylinder length=0.080948 radius=0.0059505
- link arm2-1-1: geometry visual cylinder length=0.080948 radius=0.0059505
- link arm2-1-2: geometry visual cylinder length=0.080948 radius=0.0059505
- link arm2-2-1: geometry visual cylinder length=0.080948 radius=0.0059505
- link arm2-2-2: geometry visual cylinder length=0.080948 radius=0.0059505
- link arm2-3-1: geometry visual cylinder length=0.080948 radius=0.0059505
- link arm2-3-2: geometry visual cylinder length=0.080948 radius=0.0059505
- link arm2-4-1: geometry visual cylinder length=0.080948 radius=0.0059505
- link arm2-4-2: geometry visual cylinder length=0.080948 radius=0.0059505
- link four1-1: geometry visual cylinder length=0.017 radius=0.005
- link four1-2: geometry visual cylinder length=0.017 radius=0.005
- link four1-3: geometry visual cylinder length=0.017 radius=0.005
- link four1-4: geometry visual cylinder length=0.017 radius=0.005
- link four2-1: geometry visual cylinder length=0.017 radius=0.005
- link four2-2: geometry visual cylinder length=0.017 radius=0.005
- link four2-3: geometry visual cylinder length=0.017 radius=0.005
- link four2-4: geometry visual cylinder length=0.017 radius=0.005
- link hand1-1: geometry visual cylinder length=0.034 radius=0.008
- link hand1-2: geometry visual cylinder length=0.034 radius=0.008
- link hand1-3: geometry visual cylinder length=0.034 radius=0.008
- link hand1-4: geometry visual cylinder length=0.034 radius=0.008
Joints:
- removed joint bsm1-to-bsm2
- removed joint hand2-1
- removed joint hand2-2
- removed joint hand2-3
- removed joint hand2-4
- removed joint world
- added joint arm2-3-1-to-hand1-1: type continuous, parent arm2-3-1, child hand1-1, origin xyz=0.06309 0 -0.050716 rpy=0 0 3.14159265358979323846, axis 0 1 0
- joint arm1-1: axis 0 1 0 -> (none); child arm1-1-2 -> arm1-1-1; origin xyz=0 0 0 rpy=0 0 0 -> xyz=0.06309 0 -0.050716 rpy=0 0 0; parent arm1-1-1 -> arm1-1-2
- joint arm2-1: child arm2-1-2 -> arm2-1-1; origin xyz=0 0 0 rpy=0 0 0 -> xyz=0.06309 0 -0.050716 rpy=0 0 0; parent arm2-1-1 -> arm2-1-2
- joint four1-1-to-four1-2: origin xyz=-0.017 -0.017 0 rpy=0 0 1.5708 -> xyz=-0.017 -0.017 0 rpy=0 0 1.570796326794897
- joint four1-1-to-four1-3: origin xyz=0 -0.034 0 rpy=0 0 3.1416 -> xyz=0 -0.034 0 rpy=0 0 3.14159265358979323846
- joint four1-1-to-four1-4: origin xyz=0.017 -0.017 0 rpy=0 0 -1.5708 -> xyz=0.017 -0.017 0 rpy=0 0 -1.570796326794897
- joint four2-1-to-four2-2: origin xyz=-0.017 -0.017 0 rpy=0 0 1.5708 -> xyz=-0.017 -0.017 0 rpy=0 0 1.570796326794897
- joint four2-1-to-four2-3: origin xyz=0 -0.034 0 rpy=0 0 3.1416 -> xyz=0 -0.034 0 rpy=0 0 3.14159265358979323846
- joint four2-1-to-four2-4: origin xyz=0.017 -0.017 0 rpy=0 0 -1.5708 -> xyz=0.017 -0.017 0 rpy=0 0 -1.570796326794897
- joint hand1-1: child hand1-1 -> arm1-1-2; origin xyz=-0.06309 0 0.050716 rpy=0 0 0 -> xyz=0 0.034 0 rpy=0 0 0; parent arm1-1-2 -> hand1-1
- joint wrist1-1: axis (none) -> 0 1 0; child arm1-1-1 -> four1-1; parent four1-1 -> arm1-1-1
- joint wrist1-2: axis (none) -> 0 1 0
- joint wrist1-3: axis (none) -> 0 1 0
- joint wrist1-4: axis (none) -> 0 1 0
- joint wrist2-1: axis (none) -> 0 1 0; child arm2-1-1 -> four2-1; parent four2-1 -> arm2-1-1; type continuous -> fixed
- joint wrist2-2: axis (none) -> 0 1 0
- joint wrist2-3: axis (none) -> 0 1 0
- joint wrist2-4: axis (none) -> 0 1 0

File: urdf_parser/urdfs/bsm_noladder.urdf (robot description, URDF)
Before this commit: robot BranchScissorMechanism, 33 links, 32 joints
Links:
- link hand1-1: geometry visual cylinder length=0.034 radius=0.008
- link hand1-2: geometry visual cylinder length=0.034 radius=0.008
- link hand1-3: geometry visual cylinder length=0.034 radius=0.008
- link hand1-4: geometry visual cylinder length=0.034 radius=0.008
- link hand2-1: geometry visual cylinder length=0.034 radius=0.008
- link hand2-2: geometry visual cylinder length=0.034 radius=0.008
- link hand2-3: geometry visual cylinder length=0.034 radius=0.008
- link hand2-4: geometry visual cylinder length=0.034 radius=0.008
Joints:
- removed joint arm2-3-1-to-four2-3
- removed joint four1-1-to-arm1-1-1
- removed joint four1-2-to-arm1-2-1
- removed joint four1-3-to-arm1-3-1
- removed joint four1-4-to-arm1-4-1
- removed joint four2-1-to-arm2-1-1
- removed joint four2-2-to-arm2-2-1
- removed joint four2-4-to-arm2-4-1
- added joint wrist1-1: type continuous, parent four1-1, child arm1-1-1, origin xyz=0 0 0 rpy=0 0 0
- added joint wrist1-2: type continuous, parent four1-2, child arm1-2-1, origin xyz=0 0 0 rpy=0 0 0
- added joint wrist1-3: type continuous, parent four1-3, child arm1-3-1, origin xyz=0 0 0 rpy=0 0 0
- added joint wrist1-4: type continuous, parent four1-4, child arm1-4-1, origin xyz=0 0 0 rpy=0 0 0
- added joint wrist2-1: type continuous, parent four2-1, child arm2-1-1, origin xyz=0 0 0 rpy=0 0 0
- added joint wrist2-2: type continuous, parent four2-2, child arm2-2-1, origin xyz=0 0 0 rpy=0 0 0
- added joint wrist2-3: type continuous, parent arm2-3-1, child four2-3, origin xyz=-0.06309 0 0.050716 rpy=0 0 0
- added joint wrist2-4: type continuous, parent four2-4, child arm2-4-1, origin xyz=0 0 0 rpy=0 0 0

File: urdf_parser/urdfs/scissor_2d.urdf (robot description, URDF)
Before this commit: robot DoublePendulum, 6 links, 5 joints
Links:
- added link X1_BL, mass 1; visual cylinder length=2 radius=.05
- added link X1_BR, mass 1; visual cylinder length=2 radius=.05
- added link X2_BL, mass 1; visual cylinder length=2 radius=.05
- added link X2_BR, mass 1; visual cylinder length=2 radius=.05
- added link X2_UL, mass 1; visual cylinder length=2 radius=.05
- added link X2_UR, mass 1; visual cylinder length=2 radius=.05
- link neck: geometry visual cylinder length=1 radius=.05
Joints:
- added joint X1_XJ1: type fixed, parent X1_UL, child X1_BR, origin xyz=-1.41421356 0 -1.41421356, axis 0 1 0
- added joint X1_XJ2: type fixed, parent X1_UR, child X1_BL, origin xyz=0 0 0, axis 0 1 0
- added joint X1to2L: type continuous, parent X1_BL, child X2_UL, origin xyz=1.41421356 0 -1.41421356, axis 0 1 0
- added joint X2_UJ: type continuous, parent X2_UL, child X2_UR, origin xyz=-1.41421356 0 -1.41421356, axis 0 1 0
- added joint X2_XJ1: type fixed, parent X2_UL, child X2_BR, origin xyz=-1.41421356 0 -1.41421356, axis 0 1 0
- added joint X2_XJ2: type fixed, parent X2_UR, child X2_BL, origin xyz=0 0 0, axis 0 1 0
- joint neck_base: origin xyz=0 0 -2 -> xyz=0 0 -1
