Commit message: adding constraint projection testing. works for standalone single spherical and revolute pendulums (under both translational and rotational constraint violations). constraint projection doesn't work for general URDF-parsing version

File: urdf_parser/urdfs/double_pendulum.urdf (robot description, URDF)
Before this commit: robot DoublePendulum, 3 links, 2 joints
Links:
- removed link base_link
Joints:
- removed joint shoulder
